File: Drone PCB/Drone PCB/_autosave-Drone PCB.kicad_sch (KiCad schematic)
At the start: 36 parts, among them J3 Conn_01x02_Socket, J3 Conn_01x06_Socket, J4 Conn_01x06_Pin, Q1 SI2302, Q2 SI2302, Q3 SI2302, Q4 SI2302, SW1 SW_Push, SW1 SW_SPDT, U1 AMS1117-3.3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

Commit message: PCB V1.0 layout done
Parts:
- J4: footprint Connector_PinSocket_2.54mm:PinSocket_2x03_P2.54mm_Vertical -> Connector_PinHeader_2.54mm:PinSocket_2x03_P2.54mm_Vertical
Changed lines of the file:
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@@
       (effects (font (size 1.27 1.27)) (justify right) hide)
     )
-    (property "Footprint" "Connector_PinSocket_2.54mm:PinSocket_2x03_P2.54mm_Vertical" (at 24.13 154.94 0)
+    (property "Footprint" "Connector_PinHeader_2.54mm:PinSocket_2x03_P2.54mm_Vertical" (at 24.13 154.94 0)
       (effects (font (size 1.27 1.27)) hide)
     )
